Commit message: feat: 添加多角度彩色诊断工具
- 8个视角：正面/侧面/背面/俯视/低角度/45度角
- 每个部件独立颜色标识
- 颜色图例说明
- 确认所有部件位置正确

File: robot_description/models/robotis_op2/urdf/simple_walking_robot_clean.urdf (robot description, URDF)
Before this commit: robot simple_walking_robot_clean, 8 links, 7 joints
Links:
- link body_link: geometry collision box size=0.07 0.05 0.12; visual box size=0.025 0.035 0.06
- link l_foot_link: geometry collision box size=0.08 0.04 0.015; visual box size=0.015 0.03 0.012
- link l_shin_link: geometry collision cylinder length=0.09 radius=0.014; visual capsule length=0.065 radius=0.012
- link l_thigh_link: geometry collision cylinder length=0.09 radius=0.016; visual capsule length=0.065 radius=0.014
- link r_foot_link: geometry collision box size=0.08 0.04 0.015; visual box size=0.015 0.03 0.012
- link r_shin_link: geometry collision cylinder length=0.09 radius=0.014; visual capsule length=0.065 radius=0.012
- link r_thigh_link: geometry collision cylinder length=0.09 radius=0.016; visual capsule length=0.065 radius=0.014
Joints:
- joint l_ankle_pitch: origin xyz=0 0 -0.093 -> xyz=0 0 -0.09
- joint l_hip_pitch: origin xyz=0 0.037 -0.06 -> xyz=0 0.024 -0.055
- joint l_knee: origin xyz=0 0 -0.093 -> xyz=0 0 -0.09
- joint r_ankle_pitch: origin xyz=0 0 -0.093 -> xyz=0 0 -0.09
- joint r_hip_pitch: origin xyz=0 -0.037 -0.06 -> xyz=0 -0.024 -0.055
- joint r_knee: origin xyz=0 0 -0.093 -> xyz=0 0 -0.09
